Commit message: Added gazebo control plugin

File: description/caster_wheel.xacro (robot description, xacro)
@@ -13,7 +13,17 @@
             <material name="blue"/>
         </visual>
+        <xacro:inertial_sphere mass="0.1" radius="0.05">
+            <origin xyz="0 0 0" rpy="0 0 0"/>
+        </xacro:inertial_sphere>
+        <collision>
+            <geometry>
+            <sphere radius = "0.05"/>
+            </geometry>
+        </collision>
     </link>
-    <xacro:inertial_sphere mass="0.1" radius="0.05">
-        <origin xyz="0 0 0" rpy="0 0 0"/>
-    </xacro:inertial_sphere>
+    <gazebo reference="caster_wheel">
+        <material>Gazebo/Blue</material>
+        <mu1 value="0.001"/>
+        <mu2 value="0.001"/>
+    </gazebo>
 </robot>

File: description/left_wheel.xacro (robot description, xacro)
@@ -13,9 +13,17 @@
                 <cylinder radius="0.05" length="0.04"/>
             </geometry>
+            <material name="black"/>
         </visual>
-        <material name="black"/>
+        <collision>
+            <geometry>
+                <cylinder radius="0.05" length="0.04"/>
+            </geometry>
+        </collision>
+        <xacro:inertial_cylinder mass="0.1" length="0.04" radius="0.04">
+                <origin xyz="0 0 0" rpy="0 0 0"/>
+        </xacro:inertial_cylinder>
     </link>
-    <xacro:inertial_cylinder mass="0.1" length="0.04" radius="0.04">
-        <origin xyz="0 0 0" rpy="0 0 0"/>
-    </xacro:inertial_cylinder>
+    <gazebo reference="left_wheel">
+        <material>Gazebo/Black</material>
+    </gazebo>
 </robot>

File: description/right_wheel.xacro (robot description, xacro)
@@ -13,9 +13,17 @@
                 <cylinder radius="0.05" length="0.04"/>
             </geometry>
+            <material name="black"/>
         </visual>
-    <material name="black"/>
+        <collision>
+            <geometry>
+                <cylinder radius="0.05" length="0.04"/>
+            </geometry>
+        </collision>
+        <xacro:inertial_cylinder mass="0.1" length="0.04" radius="0.04">
+            <origin xyz="0 0 0" rpy="0 0 0"/>
+        </xacro:inertial_cylinder>
     </link>
-    <xacro:inertial_cylinder mass="0.1" length="0.04" radius="0.04">
-        <origin xyz="0 0 0" rpy="0 0 0"/>
-    </xacro:inertial_cylinder>
+    <gazebo reference="right_wheel">
+        <material>Gazebo/Black</material>
+    </gazebo>
 </robot>

File: description/robot.urdf.xacro (robot description, xacro)
@@ -7,3 +7,4 @@
     <xacro:include filename="right_wheel.xacro"/>
     <xacro:include filename="caster_wheel.xacro"/>
+    <xacro:include filename="gazebo_control.xacro"/>
 </robot>

File: description/robot_core.xacro (robot description, xacro)
@@ -6,5 +6,5 @@
     <link name="chassis">
         <visual>
-            <origin  xyz="0.15 0.0 0.075" rpy="0.0 0.0 0.0"/>
+            <origin  xyz="0.15 0.0 0.075"/>
             <geometry>
                 <box size="0.3 0.3 0.15"/>
@@ -13,4 +13,5 @@
         </visual>
         <collision>
+            <origin xyz="0.15 0 0.075"/>
             <geometry>
                 <box size="0.3 0.3 0.15"/>
@@ -21,4 +22,7 @@
         </xacro:inertial_box>
     </link>
+    <gazebo reference="chassis">
+        <material>Gazebo/White</material>
+    </gazebo>
     <joint name="chassis_joint" type="fixed">
         <parent link="base_link"/>
